Commit message: Nieuwe state (srdf) en omgeving (urdf)

File: uf_robot.urdf.xacro (robot description, xacro)
@@ -202,5 +202,5 @@
   <link name="camera_stand_link">
     <visual>
-      <origin xyz="0.405 0.32 0.25" rpy="0 0 0.785398" />
+      <origin xyz="0.27 0.34 0.25" rpy="0 0 1.570796" />
       <geometry>
         <box size="0.035 0.035 0.5" />
@@ -212,5 +212,5 @@
     </inertial>
     <collision>
-      <origin xyz="0.405 0.32 0.25" rpy="0 0 0.785398" />
+      <origin xyz="0.27 0.34 0.25" rpy="0 0 1.570796" />
       <geometry>
         <box size="0.035 0.035 0.5" />
@@ -226,7 +226,7 @@
   <link name="camera_link">
     <visual>
-      <origin xyz="0.3525 0.2675 0.35" rpy="0 0 0.785398" />
-      <geometry>
-        <box size="0.105 0.105 0.06" />
+      <origin xyz="0.29 0.265 0.35" rpy="0 0 1.570796" />
+      <geometry>
+        <box size="0.11 0.11 0.07" />
       </geometry>
       <material name="LightGrey"/>
@@ -236,7 +236,7 @@
     </inertial>
     <collision>
-      <origin xyz="0.3525 0.2675 0.35" rpy="0 0 0.785398" />
-      <geometry>
-        <box size="0.105 0.105 0.06" />
+      <origin xyz="0.27 0.265 0.35" rpy="0 0 1.570796" />
+      <geometry>
+        <box size="0.11 0.11 0.07" />
       </geometry>
     </collision>
